File: docs/kicad/RPI4.kicad_sch (KiCad schematic)
At the start: 1 part, among them J1 RPI4

Commit message: hardware rewired
Changed lines of the file:
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@@
-(kicad_sch (version 20211123) (generator eeschema)
+(kicad_sch (version 20230121) (generator eeschema)
   (paper "A4")
-  (polyline (pts (xy 67.31 53.34) (xy 67.31 52.07))
-    (stroke (width 0) (type default) (color 0 0 0 0))
-  )
-  (polyline (pts (xy 55.88 54.61) (xy 55.88 63.5))
-    (stroke (width 0) (type default) (color 0 0 0 0))
-  )
-  (polyline (pts (xy 69.85 59.69) (xy 58.42 59.69))
-    (stroke (width 0) (type default) (color 0 0 0 0))
-  )
-  (polyline (pts (xy 69.85 30.48) (xy 69.85 59.69))
-    (stroke (width 0) (type default) (color 0 0 0 0))
-  )
-  (polyline (pts (xy 72.39 54.61) (xy 55.88 54.61))
-    (stroke (width 0) (type default) (color 0 0 0 0))
-  )
-  (polyline (pts (xy 64.77 60.96) (xy 62.23 62.23))
-    (stroke (width 0) (type default) (color 0 0 0 0))
-  )
-  (polyline (pts (xy 62.23 53.34) (xy 62.23 52.07))
-    (stroke (width 0) (type default) (color 0 0 0 0))
-  )
-  (polyline (pts (xy 66.04 60.96) (xy 67.31 62.23))
-    (stroke (width 0) (type default) (color 0 0 0 0))
-  )
-  (polyline (pts (xy 62.23 52.07) (xy 67.31 53.34))
-    (stroke (width 0) (type default) (color 0 0 0 0))
-  )
-  (polyline (pts (xy 58.42 30.48) (xy 69.85 30.48))
-    (stroke (width 0) (type default) (color 0 0 0 0))
-  )
-  (polyline (pts (xy 62.23 60.96) (xy 64.77 63.5))
-    (stroke (width 0) (type default) (color 0 0 0 0))
-  )
-  (polyline (pts (xy 67.31 60.96) (xy 66.04 62.23))
-    (stroke (width 0) (type default) (color 0 0 0 0))
-  )
-  (polyline (pts (xy 55.88 63.5) (xy 72.39 63.5))
-    (stroke (width 0) (type default) (color 0 0 0 0))
-  )
-  (polyline (pts (xy 72.39 63.5) (xy 72.39 54.61))
-    (stroke (width 0) (type default) (color 0 0 0 0))
-  )
-  (polyline (pts (xy 67.31 52.07) (xy 62.23 53.34))
-    (stroke (width 0) (type default) (color 0 0 0 0))
-  )
-  (polyline (pts (xy 58.42 59.69) (xy 58.42 30.48))
-    (stroke (width 0) (type default) (color 0 0 0 0))
-  )
   (image (at 64.77 53.34) (scale 1.5)
     (data
@@
     )
   )
+  (global_label "LCD RST" (shape input) (at 82.55 58.42 0) (fields_autoplaced)
+    (effects (font (size 1.27 1.27) (color 0 255 43 1)) (justify left))
+    (property "Intersheetrefs" "${INTERSHEET_REFS}" (at 92.8638 58.42 0)
+      (effects (font (size 1.27 1.27)) (justify left) hide)
+    )
+  )
+  (global_label "LCD SPI" (shape input) (at 87.63 60.96 0) (fields_autoplaced)
+    (effects (font (size 1.27 1.27) (color 0 255 43 1)) (justify left))
+    (property "Intersheetrefs" "${INTERSHEET_REFS}" (at 97.581 60.96 0)
+      (effects (font (size 1.27 1.27)) (justify left) hide)
+    )
+  )
+  (global_label "Fifo I2S" (shape input) (at 58.42 80.01 180) (fields_autoplaced)
+    (effects (font (size 1.27 1.27)) (justify right))
+    (property "Intersheetrefs" "${INTERSHEET_REFS}" (at 48.5295 80.01 0)
+      (effects (font (size 1.27 1.27)) (justify right) hide)
+    )
+  )
+  (global_label "LCD SPI" (shape input) (at 58.42 62.23 180) (fields_autoplaced)
+    (effects (font (size 1.27 1.27) (color 0 255 43 1)) (justify right))
+    (property "Intersheetrefs" "${INTERSHEET_REFS}" (at 48.469 62.23 0)
+      (effects (font (size 1.27 1.27)) (justify right) hide)
+    )
+  )
+  (global_label "IR Sensor" (shape input) (at 58.42 43.18 180) (fields_autoplaced)
+    (effects (font (size 1.27 1.27) (color 227 0 255 1)) (justify right))
+    (property "Intersheetrefs" "${INTERSHEET_REFS}" (at 46.8362 43.18 0)
+      (effects (font (size 1.27 1.27)) (justify right) hide)
+    )
+  )
+  (global_label "OUT Relay" (shape input) (at 81.28 49.53 0) (fields_autoplaced)
+    (effects (font (size 1.27 1.27) (color 227 0 255 1)) (justify left))
+    (property "Intersheetrefs" "${INTERSHEET_REFS}" (at 93.3476 49.53 0)
+      (effects (font (size 1.27 1.27)) (justify left) hide)
+    )
+  )
+  (global_label "Fifo I2S" (shape input) (at 88.9 86.36 0) (fields_autoplaced)
+    (effects (font (size 1.27 1.27)) (justify left))
+    (property "Intersheetrefs" "${INTERSHEET_REFS}" (at 98.7905 86.36 0)
+      (effects (font (size 1.27 1.27)) (justify left) hide)
+    )
+  )
+  (global_label "Rot Enc B" (shape input) (at 81.28 53.34 0) (fields_autoplaced)
+    (effects (font (size 1.27 1.27) (color 227 0 255 1)) (justify left))
+    (property "Intersheetrefs" "${INTERSHEET_REFS}" (at 93.3475 53.34 0)
+      (effects (font (size 1.27 1.27)) (justify left) hide)
+    )
+  )
+  (global_label "Rot Enc A" (shape input) (at 88.9 40.64 0) (fields_autoplaced)
+    (effects (font (size 1.27 1.27) (color 227 0 255 1)) (justify left))
+    (property "Intersheetrefs" "${INTERSHEET_REFS}" (at 100.7861 40.64 0)
+      (effects (font (size 1.27 1.27)) (justify left) hide)
+    )
+  )
+  (global_label "Fifo I2C" (shape input) (at 58.42 31.75 180) (fields_autoplaced)
+    (effects (font (size 1.27 1.27)) (justify right))
+    (property "Intersheetrefs" "${INTERSHEET_REFS}" (at 48.469 31.75 0)
+      (effects (font (size 1.27 1.27)) (justify right) hide)
+    )
+  )
+  (global_label "Fifo I2S" (shape input) (at 87.63 43.18 0) (fields_autoplaced)
+    (effects (font (size 1.27 1.27)) (justify left))
+    (property "Intersheetrefs" "${INTERSHEET_REFS}" (at 97.5205 43.18 0)
+      (effects (font (size 1.27 1.27)) (justify left) hide)
+    )
+  )
+  (global_label "PWR Relay" (shape input) (at 58.42 49.53 180) (fields_autoplaced)
+    (effects (font (size 1.27 1.27) (color 227 0 255 1)) (justify right))
+    (property "Intersheetrefs" "${INTERSHEET_REFS}" (at 45.9896 49.53 0)
+      (effects (font (size 1.27 1.27)) (justify right) hide)
+    )
+  )
+  (global_label "DAC I2C" (shape input) (at 85.09 67.31 0) (fields_autoplaced)
+    (effects (font (size 1.27 1.27) (color 0 102 255 1)) (justify left))
+    (property "Intersheetrefs" "${INTERSHEET_REFS}" (at 95.1015 67.31 0)
+      (effects (font (size 1.27 1.27)) (justify left) hide)
+    )
+  )
+  (global_label "Fifo I2C" (shape input) (at 58.42 34.29 180) (fields_autoplaced)
+    (effects (font (size 1.27 1.27)) (justify right))
+    (property "Intersheetrefs" "${INTERSHEET_REFS}" (at 48.469 34.29 0)
+      (effects (font (size 1.27 1.27)) (justify right) hide)
+    )
+  )
+  (global_label "LCD SPI" (shape input) (at 58.42 55.88 180) (fields_autoplaced)
+    (effects (font (size 1.27 1.27) (color 0 255 43 1)) (justify right))
+    (property "Intersheetrefs" "${INTERSHEET_REFS}" (at 48.469 55.88 0)
+      (effects (font (size 1.27 1.27)) (justify right) hide)
+    )
+  )
+  (global_label "DAC I2C" (shape input) (at 58.42 67.31 180) (fields_autoplaced)
+    (effects (font (size 1.27 1.27) (color 0 102 255 1)) (justify right))
+    (property "Intersheetrefs" "${INTERSHEET_REFS}" (at 48.4085 67.31 0)
+      (effects (font (size 1.27 1.27)) (justify right) hide)
+    )
+  )
+  (global_label "DAC RST" (shape input) (at 87.63 38.1 0) (fields_autoplaced)
+    (effects (font (size 1.27 1.27) (color 0 102 255 1)) (justify left))
+    (property "Intersheetrefs" "${INTERSHEET_REFS}" (at 98.0043 38.1 0)
+      (effects (font (size 1.27 1.27)) (justify left) hide)
+    )
+  )
   (symbol (lib_id "Connector:Raspberry_Pi_2_3") (at 139.7 53.34 0) (unit 1)
-    (in_bom yes) (on_board yes)
-    (property "Reference" "J1" (id 0) (at 139.7 15.7226 0))
-    (property "Value" "RPI4" (id 1) (at 139.7 18.034 0))
-    (property "Footprint" "" (id 2) (at 139.7 53.34 0)
+    (in_bom yes) (on_board yes) (dnp no)
+    (property "Reference" "J1" (at 139.7 15.7226 0)
+      (effects (font (size 1.27 1.27)))
+    )
+    (property "Value" "RPI4" (at 139.7 18.034 0)
+      (effects (font (size 1.27 1.27)))
+    )
+    (property "Footprint" "" (at 139.7 53.34 0)
       (effects (font (size 1.27 1.27)) hide)
     )
-    (property "Datasheet" "https://www.raspberrypi.org/documentation/hardware/raspberrypi/schematics/rpi_SCH_3bplus_1p0_reduced.pdf" (id 3) (at 139.7 53.34 0)
+    (property "Datasheet" "https://www.raspberrypi.org/documentation/hardware/raspberrypi/schematics/rpi_SCH_3bplus_1p0_reduced.pdf" (at 139.7 53.34 0)
       (effects (font (size 1.27 1.27)) hide)
     )
@@
     (pin "8")
     (pin "9")
+    (instances
+      (project "main_all_pages"
+        (path "/9538e4ed-27e6-4c37-b989-9859dc0d49e8/00000000-0000-0000-0000-0000601098fa"
+          (reference "J1") (unit 1)
+        )
+      )
+    )
   )
 )
