File: docs/kicad/control_board.kicad_sch (KiCad schematic)
At the start: 12 parts, among them J3 To_RPI_GPIO, J4 GPIO_To_Out_Selector_Relay, J6 POWER_OUT_TO_OLED, J7 220_IN_OUT, K1 G6S-2, Q1 BC547, SW1 RotaryEncoder_Switch, U1 TSOP312xx

Commit message: hardware rewired
Parts:
- added D1, D3: 1N4004, Diode_SMD:D_1206_3216Metric, symbol Diode:1N4004
- added J2: Drive_GPIO, Connector_PinHeader_2.54mm:PinHeader_1x02_P2.54mm_Vertical, symbol Connector:Conn_01x02_Male
- added K2, K3: G6S-2, Relay_THT:Relay_DPDT_Omron_G6S-2, symbol Relay:G6S-2
- added Q2: BC547, Package_TO_SOT_THT:TO-92_Inline, symbol Transistor_BJT:BC547
- added R1: 1K, Resistor_THT:R_Axial_DIN0207_L6.3mm_D2.5mm_P2.54mm_Vertical, symbol Device:R
Connections:
- net GPIO9 is gone; now on net GPIO23: J3.9 (Pin_9), J4.1 (Pin_1)
- net GND: now also Q2.3 (E)
- net GPIO23: now also J2.1 (Pin_1); no longer J3.8 (Pin_8)
- net GPIO18 renamed GPIO24
- new net: D1.2 (A), D3.2 (A), K2.12, K3.12, Q2.1 (C)
- new net: Q2.2 (B), R1.2
- new net 5V_SWITCH: D1.1 (K), D3.1 (K), K2.1, K3.1
