File: docs/kicad/dac.kicad_sch (KiCad schematic)
At the start: 0 parts

Commit message: hardware rewired
Changed lines of the file:
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@@
-(kicad_sch (version 20211123) (generator eeschema)
+(kicad_sch (version 20230121) (generator eeschema)
   (paper "A4")
   (wire (pts (xy 57.15 83.82) (xy 69.85 83.82))
-    (stroke (width 0) (type default) (color 0 0 0 0))
+    (stroke (width 0) (type default))
   )
   (wire (pts (xy 57.15 87.63) (xy 69.85 86.36))
-    (stroke (width 0) (type default) (color 0 0 0 0))
+    (stroke (width 0) (type default))
   )
   (wire (pts (xy 139.7 81.28) (xy 128.27 81.28))
-    (stroke (width 0) (type default) (color 0 0 0 0))
+    (stroke (width 0) (type default))
   )
   (wire (pts (xy 139.7 96.52) (xy 128.27 96.52))
-    (stroke (width 0) (type default) (color 0 0 0 0))
+    (stroke (width 0) (type default))
   )
   (wire (pts (xy 125.73 93.98) (xy 139.7 93.98))
-    (stroke (width 0) (type default) (color 0 0 0 0))
+    (stroke (width 0) (type default))
   )
   (wire (pts (xy 139.7 88.9) (xy 128.27 88.9))
-    (stroke (width 0) (type default) (color 0 0 0 0))
+    (stroke (width 0) (type default))
   )
   (wire (pts (xy 139.7 86.36) (xy 128.27 86.36))
-    (stroke (width 0) (type default) (color 0 0 0 0))
+    (stroke (width 0) (type default))
   )
   (wire (pts (xy 139.7 83.82) (xy 128.27 83.82))
-    (stroke (width 0) (type default) (color 0 0 0 0))
+    (stroke (width 0) (type default))
   )
   (wire (pts (xy 139.7 78.74) (xy 128.27 78.74))
-    (stroke (width 0) (type default) (color 0 0 0 0))
+    (stroke (width 0) (type default))
   )
   (wire (pts (xy 139.7 99.06) (xy 128.27 99.06))
-    (stroke (width 0) (type default) (color 0 0 0 0))
+    (stroke (width 0) (type default))
   )
   (wire (pts (xy 128.27 76.2) (xy 139.7 76.2))
-    (stroke (width 0) (type default) (color 0 0 0 0))
+    (stroke (width 0) (type default))
   )
   (wire (pts (xy 57.15 91.44) (xy 69.85 91.44))
-    (stroke (width 0) (type default) (color 0 0 0 0))
+    (stroke (width 0) (type default))
   )
   (image (at 99.06 86.36)
@@
     )
   )
-  (hierarchical_label "I2S_LR" (shape input) (at 139.7 78.74 0)
+  (hierarchical_label "I2S_LR" (shape input) (at 139.7 78.74 0) (fields_autoplaced)
     (effects (font (size 1.27 1.27)) (justify left))
   )
-  (hierarchical_label "I2S_DT" (shape input) (at 139.7 83.82 0)
+  (hierarchical_label "I2S_SD" (shape input) (at 139.7 83.82 0) (fields_autoplaced)
     (effects (font (size 1.27 1.27)) (justify left))
   )
-  (hierarchical_label "GPIO3" (shape input) (at 139.7 96.52 0)
+  (hierarchical_label "GPIO1" (shape input) (at 139.7 96.52 0) (fields_autoplaced)
     (effects (font (size 1.27 1.27)) (justify left))
   )
-  (hierarchical_label "I2S_BC" (shape input) (at 139.7 81.28 0)
+  (hierarchical_label "I2S_SCK" (shape input) (at 139.7 81.28 0) (fields_autoplaced)
     (effects (font (size 1.27 1.27)) (justify left))
   )
-  (hierarchical_label "I2S_V+" (shape output) (at 139.7 88.9 0)
+  (hierarchical_label "I2S_V+" (shape output) (at 139.7 88.9 0) (fields_autoplaced)
     (effects (font (size 1.27 1.27)) (justify left))
   )
-  (hierarchical_label "DAC_OUT_L" (shape output) (at 57.15 91.44 180)
+  (hierarchical_label "DAC_OUT_L" (shape output) (at 57.15 91.44 180) (fields_autoplaced)
     (effects (font (size 1.27 1.27)) (justify right))
   )
-  (hierarchical_label "DAC_OUT_GND" (shape output) (at 57.15 87.63 180)
+  (hierarchical_label "DAC_OUT_GND" (shape output) (at 57.15 87.63 180) (fields_autoplaced)
     (effects (font (size 1.27 1.27)) (justify right))
   )
-  (hierarchical_label "GPIO14" (shape input) (at 139.7 93.98 0)
+  (hierarchical_label "GPIO14" (shape input) (at 139.7 93.98 0) (fields_autoplaced)
     (effects (font (size 1.27 1.27)) (justify left))
   )
-  (hierarchical_label "I2S_MC" (shape input) (at 139.7 76.2 0)
+  (hierarchical_label "I2S_MC" (shape input) (at 139.7 76.2 0) (fields_autoplaced)
     (effects (font (size 1.27 1.27)) (justify left))
   )
-  (hierarchical_label "I2S_GND" (shape input) (at 139.7 86.36 0)
+  (hierarchical_label "I2S_GND" (shape input) (at 139.7 86.36 0) (fields_autoplaced)
     (effects (font (size 1.27 1.27)) (justify left))
   )
-  (hierarchical_label "DAC_OUT_R" (shape output) (at 57.15 83.82 180)
+  (hierarchical_label "DAC_OUT_R" (shape output) (at 57.15 83.82 180) (fields_autoplaced)
     (effects (font (size 1.27 1.27)) (justify right))
   )
-  (hierarchical_label "GPIO2" (shape input) (at 139.7 99.06 0)
+  (hierarchical_label "GPIO0" (shape input) (at 139.7 99.06 0) (fields_autoplaced)
     (effects (font (size 1.27 1.27)) (justify left))
   )
