File: docs/kicad/lcd.kicad_sch (KiCad schematic)
At the start: 2 parts, among them J13 Female_IDC_02x03_Odd_Even

Commit message: hardware rewired
Connections:
- net GPIO9: no longer names the net of J13.3 (Pin_3)
