File: docs/kicad/out_selector.kicad_sch (KiCad schematic)
At the start: 13 parts, among them J11 PWR_To_Display_BLK, J12 Drive_GPIO, J9 PWR_From_Control_Brd, K3 G6S-2, K4 G6S-2, K5 G6S-2, Q2 BC547, Q3 BC547

Commit message: hardware rewired
Parts:
- removed D3: 1N4004, Diode_SMD:D_1206_3216Metric, symbol Diode:1N4004
- removed J11: PWR_To_Display_BLK, TerminalBlock_RND:TerminalBlock_RND_205-00001_1x02_P5.00mm_Horizontal, symbol Connector:Conn_01x02_Female
- removed J9: PWR_From_Control_Brd, TerminalBlock_RND:TerminalBlock_RND_205-00001_1x02_P5.00mm_Horizontal, symbol Connector:Conn_01x02_Female
- removed K3: G6S-2, Relay_THT:Relay_DPDT_Omron_G6S-2, symbol Relay:G6S-2
- removed Q2: BC547, Package_TO_SOT_THT:TO-92_Inline, symbol Transistor_BJT:BC547
- removed R3: 1K, Resistor_THT:R_Axial_DIN0207_L6.3mm_D2.5mm_P2.54mm_Vertical, symbol Device:R
Connections:
- net GPIO9 renamed GPIO23
